Commit message: Fixed issue keyboard controller

File: urdf/main.urdf.xacro (robot description, xacro)
@@ -444,42 +444,32 @@
 	<!-- ===================================================================== -->
 	<ros2_control name="GazeboSimSystem" type="system">
-		<hardware>
-			<plugin>gz_ros2_control/GazeboSimSystem</plugin>
-		</hardware>
-		<!-- 3-wheel omni controller will command these joints -->
-		<joint name="rim_left_joint">
-			<command_interface name="velocity">
-				<param name="min">-20</param>
-				<param name="max">20</param>
-			</command_interface>
-			<state_interface name="position"/>
-			<state_interface name="velocity"/>
-		</joint>
-		<joint name="rim_right_joint">
-			<command_interface name="velocity">
-				<param name="min">-20</param>
-				<param name="max">20</param>
-			</command_interface>
-			<state_interface name="position"/>
-			<state_interface name="velocity"/>
-		</joint>
-		<joint name="rim_back_joint">
-			<command_interface name="velocity">
-				<param name="min">-20</param>
-				<param name="max">20</param>
-			</command_interface>
-			<state_interface name="position"/>
-			<state_interface name="velocity"/>
-		</joint>
-	</ros2_control>
+        <hardware>
+            <plugin>gz_ros2_control/GazeboSimSystem</plugin>
+        </hardware>
+        <joint name="rim_left_joint">
+            <command_interface name="velocity"/>
+            <state_interface name="position"/>
+            <state_interface name="velocity"/>
+        </joint>
+        <joint name="rim_right_joint">
+            <command_interface name="velocity"/>
+            <state_interface name="position"/>
+            <state_interface name="velocity"/>
+        </joint>
+        <joint name="rim_back_joint">
+            <command_interface name="velocity"/>
+            <state_interface name="position"/>
+            <state_interface name="velocity"/>
+        </joint>
+    </ros2_control>
 	<!-- gz_ros2_control plugin to connect Gazebo joints <-> ros2_control -->
 	<gazebo>
-		<plugin filename="gz_ros2_control-system" name="gz_ros2_control::GazeboSimROS2ControlPlugin">
-			<ros>
-				<!-- namespace can be overridden by launch if needed -->
-			</ros>
-			<!-- Use a parameter file that the user will create under diff/config -->
-			<parameters>$(find diff)/config/omni_wheel_drive_controller.yaml</parameters>
-		</plugin>
+	    <plugin filename="gz_ros2_control-system" name="gz_ros2_control::GazeboSimROS2ControlPlugin">
+	        <ros>
+	            <namespace>/</namespace>
+	        </ros>
+	        <parameters>$(find diff)/config/omni_wheel_drive_controller.yaml</parameters>
+	        <controller_manager_name>controller_manager</controller_manager_name>
+	    </plugin>
 	</gazebo>
 	<!-- ===================================================================== -->
@@ -545,3 +535,8 @@
         </plugin>
     </gazebo> -->
+	<gazebo>
+    	<plugin filename="libgz_ros2_control-system.so" name="gz_ros2_control::GazeboSimROS2ControlPlugin">
+        <parameters>$(find diff)/config/omni_wheel_drive_controller.yaml</parameters>
+    	</plugin>
+	</gazebo>
 </robot>

File: urdf/roller.urdf.xacro (robot description, xacro)
@@ -3,6 +3,5 @@
 	<xacro:macro
 		name="roller_macro"
-		params="parent name xyz rpy"
-	>
+		params="parent name xyz rpy">
 		<link name="roller_${name}_rim_${parent}_link">
 			<inertial>

Commit message: implement slam and nav2

File: urdf/main.urdf.xacro (robot description, xacro)
@@ -305,5 +305,5 @@
 	<link name = "laser_scanner">
 		<visual>
-		<origin xyz="0 0 0.0385" rpy="0 0 0" />
+		<origin xyz="0 0 0" rpy="0 0 0" />
 		<geometry>
 			<cylinder length="0.015" radius="0.025" />
@@ -317,5 +317,5 @@
 		<parent link = "base_link"/>
 		<child link = "laser_scanner"/>
-		<origin xyz="0 0 0.0385" rpy="0 0 0"/>
+		<origin xyz="0 0 0.077" rpy="0 0 0"/>
 	</joint>
 	<gazebo reference="laser_scanner">
